File: laser-pulse-driver/hardware/ld405-driver.kicad_pcb (KiCad board)
At the start: 4 copper layers, 160 x 100 mm, 145 parts, among them J1 9V DC IN, J2 TTL IN, J3 SET MON, J4 I MON, J5 LD OUT, J6 INTERLOCK, K1 G6K-2F-Y 5V, Q1 AO3401A, Q10 AO3400A, Q11 AO3401A, Q2 IRFR9024N, Q3 2N7002, Q4 2N7002, Q5 2N7002, Q6 AO3401A, Q7 AO3401A, Q8 2N7002, Q9 2N7002, SW1 ENABLE, U1 L78M05ABDT, U10 TLV9062, U11 LM2901, U12 74HC14, U13 74HC132, U14 74AHCT1G14, U2 REF3030, U3 TLV9062, U4 TLV9062, U5 SN74LVC1G3157, U7 OPA2192, U8 INA180A1

Commit message: laser-pulse-driver: fix relay contacts, toggle holes, REF3030 bypass
Datasheet review:
- K1 (Omron G6K-2F-Y): the normally-closed contacts are 2 and 7, not 4
  and 5. The output short-to-ground was inverted (open when disarmed,
  shorting the diode when armed). GND now goes to pins 2 and 7.
- SW1 (Dailywell 1MS1T2B4M7QES): 0.76 x 1.22 mm tab terminals need the
  datasheet's 1.85 mm holes; the footprint had 1.2 mm.
- C10 1 uF: REF30xx asks for >= 0.47 uF on its supply pin.
- Side-view LED silkscreen marks the cathode end, as is conventional.

Co-Authored-By: Claude Opus 5.5 <noreply@anthropic.com>
Claude-Session: https://claude.ai/code/session_019RAi5HuganNifeSzFvLjAT
Parts:
- C10: value 100nF -> 1uF
Connections:
- K1 pad 2: unconnected-(K1-Pad2) -> GND
- K1 pad 4: GND -> unconnected-(K1-Pad4)
- K1 pad 5: GND -> unconnected-(K1-Pad5)
- K1 pad 7: unconnected-(K1-Pad7) -> GND
