File: laser-pulse-driver/hardware/ld405-driver.kicad_pcb (KiCad board)
At the start: 4 copper layers, 160 x 100 mm, 145 parts, among them J1 9V DC IN, J2 TTL IN, J3 SET MON, J4 I MON, J5 LD OUT, J6 INTERLOCK, K1 G6K-2F-Y 5V, Q1 AO3401A, Q10 AO3400A, Q11 AO3401A, Q2 IRFR9024N, Q3 2N7002, Q4 2N7002, Q5 2N7002, Q6 AO3401A, Q7 AO3401A, Q8 2N7002, Q9 2N7002, SW1 ENABLE, U1 L78M05ABDT, U10 TLV9062, U11 LM2901, U12 74HC14, U13 74HC132, U14 74AHCT1G14, U2 REF3030, U3 TLV9062, U4 TLV9062, U5 SN74LVC1G3157, U7 OPA2192, U8 INA180A1

Commit message: laser-pulse-driver: review round 2 - Lite-On LEDs, DC jack height, toggle hole
From the review of the design-review page:
- A7: the XINGLIGHT XL-3210 datasheet contradicts itself on the cathode end
  (tape vs outline drawing). The four panel LEDs are now Lite-On LTST-S220
  (TGKT, KSKT, TBKT, KRKT), whose package and tape drawings both label the
  cathode; new footprint to Lite-On's land pattern, same polarity.
- C4: the DC-005 plug axis is 7.0 mm above the board (4.00 below the top of
  the 11 mm body), not 6.5; the rear-panel hole is moved onto it.
- C2: the toggle bushing height was never given by the drawing (6.46 is the
  lever length); measured ~6.45 mm, and the panel hole is widened to
  Ø7.4. The toggle model now has the real terminal shapes and the lever.
- A4: footprint renders put each net label beside its own pad.
- Review sections are labelled and show nuts, washers and typical mating
  plugs; regenerated board (DRC/ERC clean), fab outputs and STLs.

Co-Authored-By: Claude Opus 5.5 <noreply@anthropic.com>
Claude-Session: https://claude.ai/code/session_019RAi5HuganNifeSzFvLjAT
Parts:
- D12, D16, D3, D8: footprint ld405:LED_SideView_XL-3210 -> ld405:LED_SideView_LiteOn_LTST-S220
Routing:
- net DIS_LOOP: track 157.0 -> 161.2 mm, vias 8 -> 6
- net GND: track 102.1 -> 103.3 mm, vias 253 -> 247
